Commit message: update

File: panthera_python/Panthera-HT_description/urdf/Panthera-HT_description_follower.urdf (robot description, URDF)
Before this commit: robot Panthera-HT_description, 7 links, 6 joints
Links:
- added link tool_link
Joints:
- added joint tool_joint: type fixed, parent link6, child tool_link, origin xyz=0.165 0 0 rpy=0 0 0

File: panthera_python/Panthera-HT_description/urdf/Panthera-HT_description_leader.urdf (robot description, URDF)
Before this commit: robot Panthera-HT_description, 7 links, 6 joints
Links:
- added link tool_link
- link link6: mass 0.45 -> 0.30
Joints:
- added joint tool_joint: type fixed, parent link6, child tool_link, origin xyz=0.165 0 0 rpy=0 0 0
